File: 00_Hardware/Power.kicad_sch (KiCad schematic)
At the start: 23 parts, among them U3 FT234XD, U4 TPS560430X3FDBVR, U5 INA219BxD

Commit message: First Routing w/ output files auto-generated
Parts:
- R26: value R_Shunt -> R; symbol Device:R_Shunt -> Device:R
- U3: footprint Package_DFN_QFN:SiliconLabs_QFN-20-1EP_3x3mm_P0.5mm -> Package_DFN_QFN:DFN-12-1EP_3x3mm_P0.45mm_EP1.65x2.38mm
Connections:
- net SHUNT_IN: now also U5.8 (IN+)
- net SHUNT_OUT: now also R26.2, U5.7 (IN-); no longer R26.4
Other:
- note added: "GND BOTH ADD = 0x28"
Changed lines of the file:
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@@
+		)
+	)
+	(text "GND BOTH ADD = 0x28"
+		(exclude_from_sim no)
+		(at 255.27 78.486 0)
+		(effects
+			(font
+				(size 1.27 1.27)
+			)
 		)
 	)
@@
 	)
 	(junction
+		(at 194.31 55.88)
+		(diameter 0)
+		(color 0 0 0 0)
+	)
+	(junction
 		(at 59.69 62.23)
 		(diameter 0)
@@
 	)
 	(junction
+		(at 194.31 45.72)
+		(diameter 0)
+		(color 0 0 0 0)
+	)
+	(junction
 		(at 49.53 113.03)
 		(diameter 0)
@@
 	(wire
 		(pts
+			(xy 194.31 55.88) (xy 198.12 55.88)
+		)
+		(stroke
+			(width 0)
+			(type default)
+		)
+	)
+	(wire
+		(pts
 			(xy 198.12 48.26) (xy 223.52 48.26)
 		)
@@
 	(wire
 		(pts
+			(xy 198.12 45.72) (xy 194.31 45.72)
+		)
+		(stroke
+			(width 0)
+			(type default)
+		)
+	)
+	(wire
+		(pts
 			(xy 49.53 115.57) (xy 49.53 113.03)
 		)
@@
 	(wire
 		(pts
+			(xy 194.31 54.61) (xy 194.31 55.88)
+		)
+		(stroke
+			(width 0)
+			(type default)
+		)
+	)
+	(wire
+		(pts
 			(xy 143.51 52.07) (xy 143.51 58.42)
 		)
@@
 	(wire
 		(pts
+			(xy 198.12 48.26) (xy 198.12 45.72)
+		)
+		(stroke
+			(width 0)
+			(type default)
+		)
+	)
+	(wire
+		(pts
 			(xy 138.43 52.07) (xy 133.35 52.07)
 		)
@@
 	(wire
 		(pts
+			(xy 194.31 45.72) (xy 194.31 46.99)
+		)
+		(stroke
+			(width 0)
+			(type default)
+		)
+	)
+	(wire
+		(pts
 			(xy 62.23 156.21) (xy 77.47 156.21)
 		)
@@
 		(pts
 			(xy 102.87 148.59) (xy 109.22 148.59)
+		)
+		(stroke
+			(width 0)
+			(type default)
+		)
+	)
+	(wire
+		(pts
+			(xy 198.12 53.34) (xy 198.12 55.88)
 		)
 		(stroke
@@
 	)
 	(symbol
-		(lib_id "Device:R_Shunt")
+		(lib_id "Device:R")
 		(at 194.31 50.8 0)
 		(unit 1)
@@
 		(fields_autoplaced yes)
 		(property "Reference" "R26"
-			(at 191.77 49.5299 0)
-			(effects
-				(font
-					(size 1.27 1.27)
-				)
-				(justify right)
-			)
-		)
-		(property "Value" "R_Shunt"
-			(at 191.77 52.0699 0)
-			(effects
-				(font
-					(size 1.27 1.27)
-				)
-				(justify right)
+			(at 196.85 49.5299 0)
+			(effects
+				(font
+					(size 1.27 1.27)
+				)
+				(justify left)
+			)
+		)
+		(property "Value" "R"
+			(at 196.85 52.0699 0)
+			(effects
+				(font
+					(size 1.27 1.27)
+				)
+				(justify left)
 			)
 		)
@@
 			)
 		)
-		(property "Description" "Shunt resistor"
+		(property "Description" "Resistor"
 			(at 194.31 50.8 0)
 			(effects
@@
 		(pin "2"
 		)
-		(pin "4"
-		)
 		(pin "1"
-		)
-		(pin "3"
 		)
 		(instances
@@
 			)
 		)
-		(property "Footprint" "Package_DFN_QFN:SiliconLabs_QFN-20-1EP_3x3mm_P0.5mm"
+		(property "Footprint" "Package_DFN_QFN:DFN-12-1EP_3x3mm_P0.45mm_EP1.65x2.38mm"
 			(at 88.9 173.482 0)
 			(effects
