File: 00_Hardware/STM32G0.kicad_sch (KiCad schematic)
At the start: 26 parts, among them J4 Conn_01x04, J5 Conn_01x04, U2 STM32G030F6Px

Commit message: First Routing w/ output files auto-generated
Parts:
- added C19: 10nF, Capacitor_SMD:C_0603_1608Metric, symbol Device:C
- added R27, R28: 12k, Resistor_SMD:R_0603_1608Metric, symbol Device:R
- added R4, R5: 4.7k, Project_Footprints:R_0603_1608Metric, symbol Device:R
- added U6: TMP112xxDRL, Package_TO_SOT_SMD:SOT-563, symbol Sensor_Temperature:TMP112xxDRL
Connections:
- net +3.3V: now also R4.1, R5.1, U6.5 (V+)
- net BUTTON_1: now also U2.16 (PA9/PA11); no longer U2.7 (PA0)
- net BUTTON_2: now also U2.17 (PA10/PA12); no longer U2.8 (PA1)
- net GND: now also C19.2, R28.2, U6.2 (GND), U6.3 (ALERT), U6.4 (ADD0)
- net I2C_SCL: now also R5.2, U6.1 (SCL)
- net I2C_SDA: now also R4.2, U6.6 (SDA)
- net VBUS: now also R27.1
- new net ST_RESET: U2.8 (PA1)
- new net VSENSE: C19.1, R27.2, R28.1, U2.7 (PA0)
- no-connect marks 4 -> 2
Other:
- note added: "BOARD TEMP SENSE"
- moved on the sheet: BOOT1, R14, R15, RST1
