File: 00_Hardware/USB Stuff.kicad_sch (KiCad schematic)
At the start: 29 parts, among them J1 USB_C_Receptacle_USB2.0_16P, J2 Screw_Terminal_01x02, J3 USB_C_Receptacle_USB2.0_16P, Q1 Si7336ADP, Q2 Si7336ADP, SW1 SW_SPDT, U1 STUSB4500QTR

Commit message: First Routing w/ output files auto-generated
Parts:
- removed R4, R5: DNP, Resistor_SMD:R_0805_2012Metric, symbol Device:R
- D1, D3: footprint ESDA25W:SOT65P210X110-3N -> Project_Footprints:SOT65P210X110-3N
- D2: footprint ESDA25P35-1U1M:TVS_ESDA25P35-1U1M -> Project_Footprints:TVS_ESDA25P35-1U1M
Connections:
- net D_N: now also D3.2; no longer D3.1
- net D_P: now also D3.1; no longer D3.2
- net 1V2: no longer names the net of C5.1, U1.21 (VREG_1V2)
- net RESET renamed ST_RESET
Other:
- note added: "GND BOTH ADD = 0x28"
