File: 00_Hardware/USB_PD_JB.kicad_pcb (KiCad board)
At the start: 2 copper layers, 60 x 45 mm, 73 parts, among them J1 USB_C_Receptacle_USB2.0_16P, J2 Screw_Terminal_01x02, J3 USB_C_Receptacle_USB2.0_16P, J4 Conn_01x04, J5 Conn_01x04, Q1 Si7336ADP, Q2 Si7336ADP, SW1 SW_SPDT, U1 STUSB4500QTR, U2 STM32G030F6Px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

Commit message: First Routing w/ output files auto-generated
Parts:
- added C19: 10nF, Capacitor_SMD:C_0603_1608Metric, F.Cu at (133.0, 110.3)
- added D1: ESDA25W, Project_Footprints:SOT65P210X110-3N, F.Cu at (129.4, 97.5)
- added D2: ESDA25P35-1U1M, Project_Footprints:TVS_ESDA25P35-1U1M, F.Cu at (118.9, 90.5)
- added D3: ESDA25W, Project_Footprints:SOT65P210X110-3N, F.Cu at (129.5, 101.7)
- added D5: ESDA25P35-1U1M, Project_Footprints:TVS_ESDA25P35-1U1M, F.Cu at (169.2, 82.8)
- added R27: 12k, Resistor_SMD:R_0603_1608Metric, F.Cu at (133.0, 106.0)
- added R28: 12k, Resistor_SMD:R_0603_1608Metric, F.Cu at (133.0, 108.1)
- added U3: FT234XD, Package_DFN_QFN:DFN-12-1EP_3x3mm_P0.45mm_EP1.65x2.38mm, F.Cu at (137.6, 101.7)
- added U6: TMP112xxDRL, Package_TO_SOT_SMD:SOT-563, F.Cu at (157.8, 80.3)
- R26: value R_Shunt -> R
- R4, R5: value DNP -> 4.7k; footprint Resistor_SMD:R_0805_2012Metric -> Project_Footprints:R_0603_1608Metric
- moved R20 119.9 mm to (118.9, 123.6)
- moved R19 119.6 mm to (118.9, 120.2)
- moved R25 114.9 mm to (130.3, 91.0), turned to 180 degrees
- moved C9 109.4 mm to (134.2, 123.0)
- moved R23 106.3 mm to (132.7, 76.1)
- moved D11 106.0 mm to (130.4, 88.5)
- moved C17 103.8 mm to (139.0, 85.1)
- moved L1 101.6 mm to (134.8, 83.5), turned to -90 degrees
- moved R21 99.5 mm to (133.1, 100.5)
- moved R22 99.5 mm to (133.1, 102.9)
- moved C15 97.7 mm to (138.9, 107.1), turned to -90 degrees
- moved C10 96.6 mm to (142.5, 123.1)
- moved C13 95.3 mm to (132.0, 79.7), turned to -90 degrees
- moved R24 95.3 mm to (135.9, 76.1)
- moved C16 93.1 mm to (138.2, 81.1), turned to -90 degrees
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Connections:
- C5 pad 1: /USB Stuff/1V2 -> Net-(U1-VREG_1V2)
- R26 pad 2: Net-(U5-IN+) -> SHUNT_OUT
- R3 pad 1: RESET -> ST_RESET
- R4 pad 1: /USB Stuff/1V2 -> +3.3V
- R4 pad 2: Net-(U1-ADDR0) -> I2C_SDA
- R5 pad 1: /USB Stuff/1V2 -> +3.3V
- R5 pad 2: Net-(U1-ADDR1) -> I2C_SCL
- U1 pad 21: /USB Stuff/1V2 -> Net-(U1-VREG_1V2)
- U1 pad 6: RESET -> ST_RESET
- U2 pad 16: unconnected-(U2-PA9/PA11-Pad16) -> /STM32G0/BUTTON_1
- U2 pad 17: unconnected-(U2-PA10/PA12-Pad17) -> /STM32G0/BUTTON_2
- U2 pad 7: /STM32G0/BUTTON_1 -> /STM32G0/VSENSE
- U2 pad 8: /STM32G0/BUTTON_2 -> ST_RESET
- U5 pad 7: Net-(U5-IN-) -> SHUNT_OUT
- U5 pad 8: Net-(U5-IN+) -> SHUNT_IN
Routing:
- net +3.3V: track 0.00 -> 158.4 mm, vias 0 -> 2
- net I2C_SDA: track 0.00 -> 99.4 mm, vias 0 -> 4
- net I2C_SCL: track 0.00 -> 86.1 mm, vias 0 -> 4
- net GND: track 0.00 -> 73.4 mm, vias 0 -> 55
- net VBUS: track 0.00 -> 54.6 mm
- net SHUNT_OUT: track 0.00 -> 51.3 mm, vias 0 -> 1
- net Net-(Q1-G): track 0.00 -> 39.5 mm, vias 0 -> 4
- net /USB Stuff/CC2: track 0.00 -> 36.9 mm, vias 0 -> 3
- net SHUNT_IN: track 0.00 -> 35.7 mm
- net /STM32G0/SWDCLK/BOOT: track 0.00 -> 30.6 mm, vias 0 -> 1
- net /STM32G0/RESET: track 0.00 -> 29.5 mm, vias 0 -> 2
- net /USB Stuff/USB_OUT: track 0.00 -> 28.4 mm
- net /USB Stuff/CC1: track 0.00 -> 28.2 mm, vias 0 -> 2
- net ST_RESET: track 0.00 -> 27.6 mm, vias 0 -> 2
- net /STM32G0/SWDIO: track 0.00 -> 26.2 mm, vias 0 -> 1
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- added copper zone on F.Cu, net +3.3V
- added copper zone on F.Cu, net /USB Stuff/TERM_OUT
- added copper zone on F.Cu, net /USB Stuff/USB_OUT
- added copper zone on F.Cu, net GND
- added copper zone on In1.Cu, net GND
- added copper zone on In2.Cu, net GND
- added copper zone on F.Cu, net Net-(Q1-D)
- added copper zone on F.Cu, net Net-(U4-SW)
- added copper zone on F.Cu, net SHUNT_IN
- added copper zone on F.Cu, net SHUNT_OUT
- added copper zone on F.Cu, net VBUS
Other:
- board size 60 x 45 mm -> 60 x 64.9 mm
- copper layers 2 -> 4
- board text added: "12V"
- board text added: "15V"
- board text added: "20V"
- board text added: "3.3V GND SDA SCL"
- board text added: "3.3V GND SWD CLK"
- board text added: "5V"
- board text added: "9V"
- board text added: "BOOT"
- board text added: "INPUT"
- board text added: "INPUT VOLTAGE"
- board text added: "OTHER OUTPUT"
- board text added: "OUTPUT"
- board text added: "RESET"
- board text added: "USBC Power Board V1.0 @JBeeBK"
